File: pcb/backplane/backplane.kicad_pcb (KiCad board)
At the start: 2 copper layers, 101.6 x 101.6 mm, 102 parts, among them U1 PRPC006DAAN-RC, U10 PREC004SAAN-RC, U11 DMP3028LK3-13, U12 DMP3028LK3-13, U13 NTD4969NT4G, U14 NTD4969NT4G, U2 IFX9201SGAUMA1, U3 IFX9201SGAUMA1, U4 IFX9201SGAUMA1, U5 PREC004SAAN-RC, U6 IFX9201SGAUMA1, U7 PREC004SAAN-RC, U8 PREC004SAAN-RC, U9 PREC004SAAN-RC

Commit message: changed to a modular design
Parts:
- U2, U3, U4, U6: value IFX9201SGAUMA1 -> VAL**
- moved motorGnd3 221.2 mm to (7.62, 94.0), turned to 90 degrees
- moved motorGnd1 189.0 mm to (6.35, 24.1), turned to 90 degrees
- moved motorControlOut1 173.0 mm to (6.35, 7.62), turned to 90 degrees
- moved motorControlOut3 163.1 mm to (7.62, 77.5), turned to 90 degrees
- moved motorControlOut2 60.8 mm to (92.7, 10.2), turned to 270 degrees
- moved motorGnd2 47.5 mm to (92.7, 25.4), turned to 270 degrees
Connections:
- levelShift1 pad 5: GND -> +3V3
- levelShift2 pad 5: GND -> +3V3
- levelShift3 pad 5: GND -> +3V3
- levelShift4 pad 5: GND -> +3V3
