File: pcb/motorDriverCard/motorDriverCard.kicad_pcb (KiCad board)
At the start: 2 copper layers, 25.4 x 25.4 mm, 13 parts, among them U1 IFX9201SGAUMA1, U3 PREC004SAAN-RC, U4 TSW-104-08-T-S-RA

Commit message: updates
Parts:
- removed U4: TSW-104-08-T-S-RA, backplane:TSW-104-08-T-S-RA
- added U2: TSW-108-08-T-S-RA, backplane:TSW-108-08-T-S-RA, F.Cu at (12.7, 35.6)
- moved U1 16.5 mm to (19.1, 25.4)
- moved JST2 15.7 mm to (6.35, 22.9), turned to 0 degrees
- moved JST1 10.5 mm to (6.35, 29.2), turned to 0 degrees
- moved U3 6.48 mm to (6.35, 17.8)
Other:
- board size 25.4 x 25.4 mm -> 25.4 x 38.1 mm
Changed lines of the file:
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@@
   (general
     (thickness 1.6)
-    (drawings 6)
+    (drawings 8)
     (tracks 0)
     (zones 0)
     (modules 13)
-    (nets 18)
+    (nets 20)
   )
   (page A4)
@@
   (net 15 CSN)
   (net 16 SCK)
-  (net 17 +12V)
+  (net 17 sda)
+  (net 18 scl)
+  (net 19 +15V)
   (net_class Default "This is the default net class."
     (clearance 0.2)
@@
     (uvia_dia 0.3)
     (uvia_drill 0.1)
-    (add_net +12V)
     (add_net +14v8)
+    (add_net +15V)
     (add_net +3V3)
     (add_net +5V)
@@
     (add_net motorGnd1)
     (add_net motorPwm1)
+    (add_net scl)
+    (add_net sda)
   )
   (module backplane:865080445010 (layer B.Cu)
@@
   )
   (module backplane:B4B-XH-A (layer F.Cu)
-    (at 3.81 19.05 90)
-    (fp_text reference JST1 (at 0.5 -3.75 90) (layer F.SilkS)
-      (effects (font (size 1 1) (thickness 0.15)))
-    )
-    (fp_text value B4B-XH-A (at 0 3.75 90) (layer F.Fab)
+    (at 6.35 29.21)
+    (fp_text reference JST1 (at 0.5 -3.75) (layer F.SilkS)
+      (effects (font (size 1 1) (thickness 0.15)))
+    )
+    (fp_text value B4B-XH-A (at 0 3.75) (layer F.Fab)
       (effects (font (size 1 1) (thickness 0.15)))
     )
@@
     (fp_line (start 6.2 -1.4375) (end 6.2 1.4375) (layer F.CrtYd) (width 0.25))
     (fp_line (start 6.2 -2.875) (end 6.2 -1.4375) (layer F.CrtYd) (width 0.25))
-    (pad 4 thru_hole circle (at 3.75 0 90) (size 1.9 1.9) (drill 0.9) (layers *.Cu *.Mask)
+    (pad 4 thru_hole circle (at 3.75 0) (size 1.9 1.9) (drill 0.9) (layers *.Cu *.Mask)
       (net 4 Motor1EncoderB))
-    (pad 3 thru_hole circle (at 1.25 0 90) (size 1.9 1.9) (drill 0.9) (layers *.Cu *.Mask)
+    (pad 3 thru_hole circle (at 1.25 0) (size 1.9 1.9) (drill 0.9) (layers *.Cu *.Mask)
       (net 3 Motor1EncoderA))
-    (pad 2 thru_hole circle (at -1.25 0 90) (size 1.9 1.9) (drill 0.9) (layers *.Cu *.Mask)
+    (pad 2 thru_hole circle (at -1.25 0) (size 1.9 1.9) (drill 0.9) (layers *.Cu *.Mask)
       (net 7 +5V))
-    (pad 1 thru_hole circle (at -3.75 0 90) (size 1.9 1.9) (drill 0.9) (layers *.Cu *.Mask)
+    (pad 1 thru_hole circle (at -3.75 0) (size 1.9 1.9) (drill 0.9) (layers *.Cu *.Mask)
       (net 2 GND))
   )
   (module backplane:B4B-XH-A (layer F.Cu)
-    (at 21.59 19.05 90)
-    (fp_text reference JST2 (at 0.5 -3.75 90) (layer F.SilkS)
-      (effects (font (size 1 1) (thickness 0.15)))
-    )
-    (fp_text value B4B-XH-A (at 0 3.75 90) (layer F.Fab)
+    (at 6.35 22.86)
+    (fp_text reference JST2 (at 0.5 -3.75) (layer F.SilkS)
+      (effects (font (size 1 1) (thickness 0.15)))
+    )
+    (fp_text value B4B-XH-A (at 0 3.75) (layer F.Fab)
       (effects (font (size 1 1) (thickness 0.15)))
     )
@@
     (fp_line (start -6.2 -1.4375) (end -4.65 -2.875) (layer F.SilkS) (width 0.25))
     (fp_line (start -4.65 -2.875) (end 6.2 -2.875) (layer F.SilkS) (width 0.25))
-    (pad 1 thru_hole circle (at -3.75 0 90) (size 1.9 1.9) (drill 0.9) (layers *.Cu *.Mask)
+    (pad 1 thru_hole circle (at -3.75 0) (size 1.9 1.9) (drill 0.9) (layers *.Cu *.Mask)
       (net 7 +5V))
-    (pad 2 thru_hole circle (at -1.25 0 90) (size 1.9 1.9) (drill 0.9) (layers *.Cu *.Mask)
-      (net 2 GND))
-    (pad 3 thru_hole circle (at 1.25 0 90) (size 1.9 1.9) (drill 0.9) (layers *.Cu *.Mask)
+    (pad 2 thru_hole circle (at -1.25 0) (size 1.9 1.9) (drill 0.9) (layers *.Cu *.Mask)
+      (net 2 GND))
+    (pad 3 thru_hole circle (at 1.25 0) (size 1.9 1.9) (drill 0.9) (layers *.Cu *.Mask)
       (net 3 Motor1EncoderA))
-    (pad 4 thru_hole circle (at 3.75 0 90) (size 1.9 1.9) (drill 0.9) (layers *.Cu *.Mask)
+    (pad 4 thru_hole circle (at 3.75 0) (size 1.9 1.9) (drill 0.9) (layers *.Cu *.Mask)
       (net 4 Motor1EncoderB))
   )
@@
   )
   (module backplane:IFX9201SGAUMA1 (layer F.Cu)
-    (at 12.7 10.16 90)
+    (at 19.05 25.4 90)
     (attr smd)
     (fp_text reference U1 (at 0 -5.08 90) (layer F.SilkS)
@@
   )
   (module backplane:PREC004SAAN-RC (layer F.Cu)
-    (at 12.7 19.05)
+    (at 6.35 17.78)
     (fp_text reference U3 (at 0 -4.445) (layer F.SilkS)
       (effects (font (size 1 1) (thickness 0.15)))
@@
       (net 16 SCK))
   )
-  (module backplane:TSW-104-08-T-S-RA (layer F.Cu)
-    (at 12.7 22.86 180)
-    (fp_text reference U4 (at 0 -12.7 180) (layer F.SilkS)
-      (effects (font (size 1 1) (thickness 0.15)))
-    )
-    (fp_text value TSW-104-08-T-S-RA (at 0 -10.795 180) (layer F.Fab)
-      (effects (font (size 1 1) (thickness 0.15)))
-    )
-    (fp_line (start 5.08 -1.27) (end 5.08 1.27) (layer F.SilkS) (width 0.25))
-    (fp_line (start 5.08 1.27) (end -5.08 1.27) (layer F.SilkS) (width 0.25))
-    (fp_line (start -5.08 1.27) (end -5.08 -0.635) (layer F.SilkS) (width 0.25))
-    (fp_line (start -5.08 -0.635) (end -4.445 -1.27) (layer F.SilkS) (width 0.25))
-    (fp_line (start -4.445 -1.27) (end 5.08 -1.27) (layer F.SilkS) (width 0.25))
-    (fp_line (start -5.335 0) (end -5.335 -9.88) (layer F.CrtYd) (width 0.25))
-    (fp_line (start -5.335 -9.88) (end 5.335 -9.88) (layer F.CrtYd) (width 0.25))
-    (fp_line (start 5.335 0) (end 5.335 -9.88) (layer F.CrtYd) (width 0.25))
-    (fp_line (start -5.335 0) (end -5.335 1.27) (layer F.CrtYd) (width 0.25))
-    (fp_line (start -5.335 1.27) (end 5.335 1.27) (layer F.CrtYd) (width 0.25))
-    (fp_line (start 5.335 1.27) (end 5.335 0) (layer F.CrtYd) (width 0.25))
-    (pad 1 thru_hole circle (at -3.81 0 180) (size 2.02 2.02) (drill 1.02) (layers *.Cu *.Mask)
-      (net 17 +12V))
-    (pad 2 thru_hole circle (at -1.27 0 180) (size 2.02 2.02) (drill 1.02) (layers *.Cu *.Mask)
+  (module backplane:TSW-108-08-T-S-RA (layer F.Cu)
+    (at 12.7 35.56 180)
+    (fp_text reference U2 (at 0 -12.7 180) (layer F.SilkS)
+      (effects (font (size 1 1) (thickness 0.15)))
+    )
+    (fp_text value TSW-108-08-T-S-RA (at 0 -10.795 180) (layer F.Fab)
+      (effects (font (size 1 1) (thickness 0.15)))
+    )
+    (fp_line (start 0 1.27) (end -10.16 1.27) (layer F.SilkS) (width 0.25))
+    (fp_line (start -10.16 1.27) (end -10.16 -0.635) (layer F.SilkS) (width 0.25))
+    (fp_line (start -10.16 -0.635) (end -9.525 -1.27) (layer F.SilkS) (width 0.25))
+    (fp_line (start -9.525 -1.27) (end 0 -1.27) (layer F.SilkS) (width 0.25))
+    (fp_line (start -10.415 0) (end -10.415 -9.88) (layer F.CrtYd) (width 0.25))
+    (fp_line (start -10.415 -9.88) (end 10.415 -9.88) (layer F.CrtYd) (width 0.25))
+    (fp_line (start 10.415 0) (end 10.415 -9.88) (layer F.CrtYd) (width 0.25))
+    (fp_line (start 0 -1.27) (end 10.16 -1.27) (layer F.SilkS) (width 0.25))
+    (fp_line (start 10.16 -1.27) (end 10.16 1.27) (layer F.SilkS) (width 0.25))
+    (fp_line (start 10.16 1.27) (end 0 1.27) (layer F.SilkS) (width 0.25))
+    (fp_line (start -10.415 0) (end -10.415 1.27) (layer F.CrtYd) (width 0.25))
+    (fp_line (start -10.415 1.27) (end 10.415 1.27) (layer F.CrtYd) (width 0.25))
+    (fp_line (start 10.415 1.27) (end 10.415 0) (layer F.CrtYd) (width 0.25))
+    (pad 1 thru_hole circle (at -8.89 0 180) (size 2.02 2.02) (drill 1.02) (layers *.Cu *.Mask)
+      (net 17 sda))
+    (pad 2 thru_hole circle (at -6.35 0 180) (size 2.02 2.02) (drill 1.02) (layers *.Cu *.Mask)
+      (net 18 scl))
+    (pad 3 thru_hole circle (at -3.81 0 180) (size 2.02 2.02) (drill 1.02) (layers *.Cu *.Mask)
+      (net 19 +15V))
+    (pad 4 thru_hole circle (at -1.27 0 180) (size 2.02 2.02) (drill 1.02) (layers *.Cu *.Mask)
+      (net 19 +15V))
+    (pad 5 thru_hole circle (at 1.27 0 180) (size 2.02 2.02) (drill 1.02) (layers *.Cu *.Mask)
       (net 7 +5V))
-    (pad 3 thru_hole circle (at 1.27 0 180) (size 2.02 2.02) (drill 1.02) (layers *.Cu *.Mask)
+    (pad 6 thru_hole circle (at 3.81 0 180) (size 2.02 2.02) (drill 1.02) (layers *.Cu *.Mask)
       (net 8 +3V3))
-    (pad 4 thru_hole circle (at 3.81 0 180) (size 2.02 2.02) (drill 1.02) (layers *.Cu *.Mask)
-      (net 2 GND))
-  )
+    (pad 7 thru_hole circle (at 6.35 0 180) (size 2.02 2.02) (drill 1.02) (layers *.Cu *.Mask)
+      (net 2 GND))
+    (pad 8 thru_hole circle (at 8.89 0 180) (size 2.02 2.02) (drill 1.02) (layers *.Cu *.Mask)
+      (net 2 GND))
+  )
+  (gr_line (start 25.4 38.1) (end 25.4 25.4) (layer Edge.Cuts) (width 0.15))
+  (gr_line (start 0 38.1) (end 25.4 38.1) (layer Edge.Cuts) (width 0.15))
+  (gr_line (start 0 25.4) (end 0 38.1) (layer Edge.Cuts) (width 0.15))
   (gr_line (start 0 12.7) (end 25.4 12.7) (layer F.SilkS) (width 0.2))
   (gr_line (start 12.7 0) (end 12.7 25.4) (layer F.SilkS) (width 0.2))
   (gr_line (start 25.4 0) (end 25.4 25.4) (layer Edge.Cuts) (width 0.15))
   (gr_line (start 0 0) (end 0 25.4) (layer Edge.Cuts) (width 0.15))
-  (gr_line (start 0 25.4) (end 25.4 25.4) (layer Edge.Cuts) (width 0.15))
   (gr_line (start 0 0) (end 25.4 0) (layer Edge.Cuts) (width 0.15))
 )

Commit message: updates
Parts:
- removed encoderpins1, encoderpins2, motorControl1: PREC002SAAN-RC, backplane:PREC002SAAN-RC
- C1, C3, levelShift2: moved to F.Cu
- U2: value TSW-108-08-T-S-RA -> PEC07DBBN; footprint backplane:TSW-108-08-T-S-RA -> backplane:PEC07DBBN
- moved C3 28.1 mm to (47.0, 3.81), turned to 270 degrees
- moved levelShift2 20.9 mm to (39.4, 5.08)
- moved JST1 20.1 mm to (17.8, 12.7), turned to 90 degrees
- moved C1 19.9 mm to (3.81, 25.4), turned to 270 degrees
- moved JST2 10.5 mm to (8.89, 12.7), turned to 90 degrees
- moved U3 6.35 mm to (2.54, 12.7), turned to 90 degrees
- moved U1 2.84 mm to (16.5, 24.1), turned to 0 degrees
Connections:
- U2 pad 1: sda -> GND
- U2 pad 2: scl -> GND
- U2 pad 3: +15V -> +3V3
- U2 pad 4: +15V -> +5V
- U2 pad 5: +5V -> +15V
- U2 pad 6: +3V3 -> +15V
- U2 pad 7: GND -> sda
- U2 pad 8: GND -> Motor1EncoderA_3v3

Commit message: motordriver finished
Parts:
- removed JST1: B4B-XH-A, backplane:B4B-XH-A
- removed U1: IFX9201SGAUMA1, backplane:IFX9201SGAUMA1
- added Driver1: IFX9201SGAUMA1, backplane:IFX9201SGAUMA1, F.Cu at (12.7, 14.5)
- C1, C3: moved to B.Cu
- moved C3 43.4 mm to (4.57, 13.2), turned to 90 degrees
- moved Shift1 29.0 mm to (14.7, 20.4), turned to 90 degrees
- moved Encoder1 13.4 mm to (13.2, 25.4), turned to 0 degrees
- moved SPI1 11.3 mm to (12.7, 7.75), turned to 0 degrees
- moved C1 2.55 mm to (4.06, 22.9)
- moved CardConnector1 1.27 mm to (12.7, 34.3)
- renumbered U2 to CardConnector1, JST2 to Encoder1, motorGnd1 to MotorGnd1, motorControlOut1 to MotorOut1, U3 to SPI1, levelShift2 to Shift1
Connections:
- C1 pad 1: +14v8 -> +15V
- C3 pad 1: +14v8 -> +15V
- CardConnector1 pad 1: GND -> sda
- CardConnector1 pad 10: Motor1EncoderB_3v3 -> Motor1EncoderA_3v3
- CardConnector1 pad 11: motorPwm1 -> motorDir1
- CardConnector1 pad 13: motorDir1 -> motorPwm1
- CardConnector1 pad 2: GND -> scl
- CardConnector1 pad 7: sda -> GND
- CardConnector1 pad 8: Motor1EncoderA_3v3 -> Motor1EncoderB_3v3
- CardConnector1 pad 9: scl -> GND
Routing:
- net motorPwm1: track 0.00 -> 44.4 mm, vias 0 -> 1
- net motorDir1: track 0.00 -> 34.9 mm, vias 0 -> 1
- net Motor1EncoderB_3v3: track 0.00 -> 21.0 mm
- net Motor1EncoderA_3v3: track 0.00 -> 20.9 mm
- net Motor1EncoderB: track 0.00 -> 19.6 mm
- net mcuSI: track 0.00 -> 14.7 mm, vias 0 -> 1
- net Motor1EncoderA: track 0.00 -> 14.3 mm
- net CSN: track 0.00 -> 12.0 mm, vias 0 -> 1
- net mcuSO: track 0.00 -> 9.00 mm, vias 0 -> 1
- net SCK: track 0.00 -> 6.82 mm, vias 0 -> 1
- net +3V3: track 0.00 -> 3.87 mm, vias 0 -> 3
- net GND: track 0.00 -> 3.31 mm, vias 0 -> 20
- net +5V: track 0.00 -> 0.92 mm, vias 0 -> 1
- net +15V: vias 0 -> 7
- added copper zone on 15V, net +15V
- added copper zone on F.Cu, net +15V
- added copper zone on 3V3, net +3V3
- added copper zone on 5V, net +5V
- added copper zone on F.Cu, net GND
- added copper zone on GND, net GND
- added copper zone on F.Cu, net motorControlOut1
- added copper zone on F.Cu, net motorGnd1
Other:
- copper layers 2 -> 6
- board text added: "Reaper Tech"
