File: pcb/motorDriverCard/motorDriverCard.sch (KiCad schematic (older format))
At the start: 13 parts, among them U1 IFX9201SGAUMA1, U3 PREC004SAAN-RC, U4 TSW-104-08-T-S-RA

Commit message: updates
Parts:
- removed U4: TSW-104-08-T-S-RA, backplane:TSW-104-08-T-S-RA, symbol backplane_Library:TSW-104-08-T-S-RA
- added U2: TSW-108-08-T-S-RA, backplane:TSW-108-08-T-S-RA, symbol backplane_Library:TSW-108-08-T-S-RA
Connections:
- net +3V3: now also U2.6 (F)
- net +5V: now also U2.5 (E)
- net GND: now also U2.7 (G), U2.8 (H)
- new net +15V: U2.3 (C), U2.4 (D)
- new net scl: U2.2 (B)
- new net sda: U2.1 (A)
Changed lines of the file:
@@
 Wire Wire Line
 	7000 1750 7000 1950
-$Comp
-L power:+3.3V #PWR028
-U 1 1 5C79A90C
-P 1550 7200
-F 0 "#PWR028" H 1550 7050 50  0001 C CNN
-F 1 "+3.3V" H 1565 7373 50  0000 C CNN
-F 2 "" H 1550 7200 50  0001 C CNN
-F 3 "" H 1550 7200 50  0001 C CNN
-	1    1550 7200
-	-1   0    0    1
-$EndComp
-$Comp
-L power:+5V #PWR027
-U 1 1 5C79A995
-P 1350 7200
-F 0 "#PWR027" H 1350 7050 50  0001 C CNN
-F 1 "+5V" H 1365 7373 50  0000 C CNN
-F 2 "" H 1350 7200 50  0001 C CNN
-F 3 "" H 1350 7200 50  0001 C CNN
-	1    1350 7200
-	-1   0    0    1
-$EndComp
-$Comp
-L power:+12V #PWR026
-U 1 1 5C79AA1E
-P 1150 7200
-F 0 "#PWR026" H 1150 7050 50  0001 C CNN
-F 1 "+12V" H 1165 7373 50  0000 C CNN
-F 2 "" H 1150 7200 50  0001 C CNN
-F 3 "" H 1150 7200 50  0001 C CNN
-	1    1150 7200
-	-1   0    0    1
-$EndComp
-$Comp
-L power:GND #PWR025
-U 1 1 5C79E2E3
-P 1750 7200
-F 0 "#PWR025" H 1750 6950 50  0001 C CNN
-F 1 "GND" H 1755 7027 50  0000 C CNN
-F 2 "" H 1750 7200 50  0001 C CNN
-F 3 "" H 1750 7200 50  0001 C CNN
-	1    1750 7200
-	1    0    0    -1
-$EndComp
-$Comp
-L backplane_Library:TSW-104-08-T-S-RA U4
-U 1 1 5CD5F480
-P 1450 6800
-F 0 "U4" H 1728 6715 50  0000 L CNN
-F 1 "TSW-104-08-T-S-RA" H 1728 6624 50  0000 L CNN
-F 2 "backplane:TSW-104-08-T-S-RA" H 1450 6850 50  0001 C CNN
-F 3 "" H 1450 6850 50  0001 C CNN
-	1    1450 6800
-	1    0    0    -1
-$EndComp
-Wire Wire Line
-	1750 7200 1750 7050
-Wire Wire Line
-	1750 7050 1600 7050
-Wire Wire Line
-	1550 7200 1550 7100
-Wire Wire Line
-	1550 7100 1500 7100
-Wire Wire Line
-	1500 7100 1500 7050
-Wire Wire Line
-	1350 7200 1350 7100
-Wire Wire Line
-	1350 7100 1400 7100
-Wire Wire Line
-	1400 7100 1400 7050
-Wire Wire Line
-	1150 7200 1150 7050
-Wire Wire Line
-	1150 7050 1300 7050
 Wire Wire Line
 	1150 1650 1150 1550
@@
 Text Notes 950  6700 0    50   ~ 0
 power to card from backplane
+$Comp
+L backplane_Library:TSW-108-08-T-S-RA U2
+U 1 1 5C555696
+P 1500 6850
+F 0 "U2" H 1495 7015 50  0000 C CNN
+F 1 "TSW-108-08-T-S-RA" H 1495 6924 50  0000 C CNN
+F 2 "backplane:TSW-108-08-T-S-RA" H 1450 7100 50  0001 C CNN
+F 3 "" H 1450 7100 50  0001 C CNN
+	1    1500 6850
+	1    0    0    -1
+$EndComp
+$Comp
+L power:+15V #PWR0101
+U 1 1 5C555725
+P 1450 7400
+F 0 "#PWR0101" H 1450 7250 50  0001 C CNN
+F 1 "+15V" H 1465 7573 50  0000 C CNN
+F 2 "" H 1450 7400 50  0001 C CNN
+F 3 "" H 1450 7400 50  0001 C CNN
+	1    1450 7400
+	-1   0    0    1
+$EndComp
+$Comp
+L power:+3.3V #PWR0102
+U 1 1 5C55591F
+P 1850 7400
+F 0 "#PWR0102" H 1850 7250 50  0001 C CNN
+F 1 "+3.3V" H 1865 7573 50  0000 C CNN
+F 2 "" H 1850 7400 50  0001 C CNN
+F 3 "" H 1850 7400 50  0001 C CNN
+	1    1850 7400
+	-1   0    0    1
+$EndComp
+$Comp
+L power:+5V #PWR0103
+U 1 1 5C555925
+P 1650 7400
+F 0 "#PWR0103" H 1650 7250 50  0001 C CNN
+F 1 "+5V" H 1665 7573 50  0000 C CNN
+F 2 "" H 1650 7400 50  0001 C CNN
+F 3 "" H 1650 7400 50  0001 C CNN
+	1    1650 7400
+	-1   0    0    1
+$EndComp
+$Comp
+L power:GND #PWR0104
+U 1 1 5C555931
+P 2050 7400
+F 0 "#PWR0104" H 2050 7150 50  0001 C CNN
+F 1 "GND" H 2055 7227 50  0000 C CNN
+F 2 "" H 2050 7400 50  0001 C CNN
+F 3 "" H 2050 7400 50  0001 C CNN
+	1    2050 7400
+	1    0    0    -1
+$EndComp
+$Comp
+L power:GND #PWR0105
+U 1 1 5C556C8F
+P 2250 7400
+F 0 "#PWR0105" H 2250 7150 50  0001 C CNN
+F 1 "GND" H 2255 7227 50  0000 C CNN
+F 2 "" H 2250 7400 50  0001 C CNN
+F 3 "" H 2250 7400 50  0001 C CNN
+	1    2250 7400
+	1    0    0    -1
+$EndComp
+$Comp
+L power:+15V #PWR0106
+U 1 1 5C55ED33
+P 1250 7400
+F 0 "#PWR0106" H 1250 7250 50  0001 C CNN
+F 1 "+15V" H 1265 7573 50  0000 C CNN
+F 2 "" H 1250 7400 50  0001 C CNN
+F 3 "" H 1250 7400 50  0001 C CNN
+	1    1250 7400
+	-1   0    0    1
+$EndComp
+Wire Wire Line
+	2250 7400 2250 7100
+Wire Wire Line
+	2250 7100 1850 7100
+Wire Wire Line
+	2050 7400 2050 7200
+Wire Wire Line
+	2050 7200 1750 7200
+Wire Wire Line
+	1750 7200 1750 7100
+Wire Wire Line
+	1850 7400 1850 7250
+Wire Wire Line
+	1850 7250 1650 7250
+Wire Wire Line
+	1650 7250 1650 7100
+Wire Wire Line
+	1650 7400 1550 7400
+Wire Wire Line
+	1550 7400 1550 7100
+Wire Wire Line
+	1450 7400 1450 7100
+Wire Wire Line
+	1250 7400 1250 7250
+Wire Wire Line
+	1250 7250 1350 7250
+Wire Wire Line
+	1350 7250 1350 7100
+Text GLabel 950  7300 3    50   Input ~ 0
+sda
+Wire Wire Line
+	950  7300 950  7100
+Wire Wire Line
+	950  7100 1150 7100
+Text GLabel 1100 7300 3    50   Input ~ 0
+scl
+Wire Wire Line
+	1100 7300 1100 7150
+Wire Wire Line
+	1100 7150 1250 7150
+Wire Wire Line
+	1250 7150 1250 7100
 $EndSCHEMATC

Commit message: updates
Parts:
- removed U2: TSW-108-08-T-S-RA, backplane:TSW-108-08-T-S-RA, symbol backplane_Library:TSW-108-08-T-S-RA
- removed encoderpins1, encoderpins2, motorControl1: PREC002SAAN-RC, backplane:PREC002SAAN-RC, symbol motorDriverCard-rescue:PREC002SAAN-RC-backplane_Library-backplane-rescue
- added U2: PEC07DBBN, backplane:PEC07DBBN, symbol backplane_Library:PEC07DBBN
Connections:
- net +15V: now also U2.5 (E), U2.6 (F)
- net +3V3: now also U2.3 (C)
- net +5V: now also U2.4 (D)
- net GND: now also U2.1 (A), U2.2 (B)
- net Motor1EncoderA: now also U2.12 (L)
- net Motor1EncoderA_3v3: now also U2.8 (H)
- net Motor1EncoderB: now also U2.14 (N)
- net Motor1EncoderB_3v3: now also U2.10 (J)
- net motorDir1: now also U2.13 (M)
- net motorPwm1: now also U2.11 (K)
- net scl: now also U2.9 (I)
- net sda: now also U2.7 (G)
Other:
- note removed: "Encoder pins to mcu"
- moved on the sheet: C1, C3, U1

Commit message: motordriver finished
Parts:
- removed JST1: B4B-XH-A, backplane:B4B-XH-A, symbol motorDriverCard-rescue:B4B-XH-A-backplane_Library-backplane-rescue
- renumbered U2 to CardConnector1, U1 to Driver1, JST2 to Encoder1, motorGnd1 to MotorGnd1, motorControlOut1 to MotorOut1, U3 to SPI1, levelShift2 to Shift1
Connections:
- net +14v8 is gone; now on net +15V: C1.1, C3.1, Driver1.4 (VS)
- net GND: now also CardConnector1.7 (G), CardConnector1.9 (I); no longer CardConnector1.1 (A), CardConnector1.2 (B)
- net Motor1EncoderA_3v3: now also CardConnector1.10 (J); no longer CardConnector1.8 (H)
- net Motor1EncoderB_3v3: now also CardConnector1.8 (H); no longer CardConnector1.10 (J)
- net motorDir1: now also CardConnector1.11 (K); no longer CardConnector1.13 (M)
- net motorPwm1: now also CardConnector1.13 (M); no longer CardConnector1.11 (K)
- net scl: now also CardConnector1.2 (B); no longer CardConnector1.9 (I)
- net sda: now also CardConnector1.1 (A); no longer CardConnector1.7 (G)
Other:
- note removed: "jst connectors that support textrix and rev motors"
- moved on the sheet: SPI1, Shift1
